Commit message: prefix versions of gazebo and transmission macros

File: ur_description/urdf/ur10.gazebo.xacro (robot description, xacro)
@@ -4,30 +4,30 @@
        xmlns:interface="http://playerstage.sourceforge.net/gazebo/xmlschema/#interface"
        xmlns:xacro="http://ros.org/wiki/xacro">
-	<xacro:macro name="ur10_arm_gazebo" params="name">
-		<gazebo reference="${name}_base_link">
+	<xacro:macro name="ur10_arm_gazebo" params="prefix">
+		<gazebo reference="${prefix}base_link">
 			<material value="Gazebo/Grey" />
 			<turnGravityOff>false</turnGravityOff>
 		</gazebo>
-		<gazebo reference="${name}_shoulder_pan_link">
+		<gazebo reference="${prefix}shoulder_pan_link">
 			<material value="Gazebo/Blue " />
 			<turnGravityOff>false</turnGravityOff>
 		</gazebo>
-		<gazebo reference="${name}_shoulder_lift_link">
+		<gazebo reference="${prefix}shoulder_lift_link">
 			<material value="Gazebo/Grey" />
 			<turnGravityOff>false</turnGravityOff>
 		</gazebo>
-		<gazebo reference="${name}_elbow_link">
+		<gazebo reference="${prefix}elbow_link">
 			<material value="Gazebo/Blue " />
 			<turnGravityOff>false</turnGravityOff>
 		</gazebo>
-		<gazebo reference="${name}_wrist_1_link">
+		<gazebo reference="${prefix}wrist_1_link">
 			<material value="Gazebo/Grey" />
 			<turnGravityOff>false</turnGravityOff>
 		</gazebo>
-		<gazebo reference="${name}_wrist_2_link">
+		<gazebo reference="${prefix}wrist_2_link">
 			<material value="Gazebo/Blue " />
 			<turnGravityOff>false</turnGravityOff>
 		</gazebo>
-		<gazebo reference="${name}_wrist_1_link">
+		<gazebo reference="${prefix}wrist_1_link">
 			<material value="Gazebo/Grey" />
 			<turnGravityOff>false</turnGravityOff>

File: ur_description/urdf/ur10.transmission.xacro (robot description, xacro)
@@ -4,33 +4,33 @@
        xmlns:interface="http://playerstage.sourceforge.net/gazebo/xmlschema/#interface"
        xmlns:xacro="http://ros.org/wiki/xacro">
-	<xacro:macro name="ur10_arm_transmission" params="name">
+	<xacro:macro name="ur10_arm_transmission" params="prefix">
 		<transmission name="shoulder_pan_trans" type="pr2_mechanism_model/SimpleTransmission">
 			<actuator name="shoulder_pan_motor"/>
-			<joint name="${name}_shoulder_pan_joint"/>
+			<joint name="${prefix}shoulder_pan_joint"/>
 			<mechanicalReduction>1</mechanicalReduction>
 		</transmission>
 		<transmission name="shoulder_lift_trans" type="pr2_mechanism_model/SimpleTransmission">
 			<actuator name="shoulder_lift_motor"/>
-			<joint name="${name}_shoulder_lift_joint"/>
+			<joint name="${prefix}shoulder_lift_joint"/>
 			<mechanicalReduction>1</mechanicalReduction>
 		</transmission>
 		<transmission name="elbow_trans" type="pr2_mechanism_model/SimpleTransmission">
 			<actuator name="elbow_motor"/>
-			<joint name="${name}_elbow_joint"/>
+			<joint name="${prefix}elbow_joint"/>
 			<mechanicalReduction>1</mechanicalReduction>
 		</transmission>
 		<transmission name="wrist_1_trans" type="pr2_mechanism_model/SimpleTransmission">
 			<actuator name="wrist_1_motor"/>
-			<joint name="${name}_wrist_1_joint"/>
+			<joint name="${prefix}wrist_1_joint"/>
 			<mechanicalReduction>1</mechanicalReduction>
 		</transmission>
 		<transmission name="wrist_2_trans" type="pr2_mechanism_model/SimpleTransmission">
 			<actuator name="wrist_2_motor"/>
-			<joint name="${name}_wrist_2_joint"/>
+			<joint name="${prefix}wrist_2_joint"/>
 			<mechanicalReduction>1</mechanicalReduction>
 		</transmission>
 		<transmission name="wrist_3_trans" type="pr2_mechanism_model/SimpleTransmission">
 			<actuator name="wrist_3_motor"/>
-			<joint name="${name}_wrist_3_joint"/>
+			<joint name="${prefix}wrist_3_joint"/>
 			<mechanicalReduction>1</mechanicalReduction>
 		</transmission>

File: ur_description/urdf/ur10.urdf.xacro (robot description, xacro)
@@ -226,6 +226,6 @@
     </inertial>
   </link>
-  <xacro:ur10_arm_transmission name="${prefix}" />
-  <xacro:ur10_arm_gazebo name="${prefix}" />
+  <xacro:ur10_arm_transmission prefix="${prefix}" />
+  <xacro:ur10_arm_gazebo prefix="${prefix}" />
   </xacro:macro>
 </robot>
