Commit message: merged ur10 description from GT

File: ur_description/urdf/ur10.urdf.xacro (robot description, xacro)
@@ -7,54 +7,69 @@
   <include filename="$(find ur_description)/urdf/ur10.gazebo.xacro" />
   <include filename="$(find ur_description)/urdf/materials.urdf.xacro" />
+<!--
+DH for UR5:
+a = [0.00000, -0.42500, -0.39225,  0.00000,  0.00000,  0.0000]
+d = [0.089159,  0.00000,  0.00000,  0.10915,  0.09465,  0.0823]
+alpha = [ 1.570796327, 0, 0, 1.570796327, -1.570796327, 0 ]
+q_home_offset = [0, -1.570796327, 0, -1.570796327, 0, 0]
+joint_direction = [-1, -1, 1, 1, 1, 1]
+DH for UR10:
+a = [0.000, -0.612, -0.5723, 0.000000, 0.0000, 0.0000]
+d = [0.1273,  0.000,  0.0000, 0.163941, 0.1157, 0.0922]
+alpha = [ 1.570796327, 0, 0, 1.570796327, -1.570796327, 0 ]
+q_home_offset = [0, -1.570796327, 0, -1.570796327, 0, 0]
+joint_direction = [1, 1, -1, 1, 1, 1]
+Mass for UR5:
+mass = [3.7000, 8.3930, 2.2750, 1.2190, 1.2190, 0.1879]
+center_of_mass = [ [0, -0.02561, 0.00193], [0.2125, 0, 0.11336], [0.11993, 0.0, 0.0265], [0, -0.0018, 0.01634], [0, 0.0018,0.01634], [0, 0, -0.001159] ]
+Mass for UR10:
+mass = [7.778, 12.930, 3.87, 1.96, 1.96, 0.202]
+center_of_mass = [ [0.00008, -0.037, 0.00244], [0.38757, 0.00001, 0.15061], [0.1984, -0.00012, 0.06112], [-0.00021, -0.00112, 0.02269], [-0.00021, 0.00112, 0.002269], [-0.00149, 0, -0.001156] ]
+-->
   <property name="pi" value="3.14159265" />
-  <!-- Inertia parameters -->
-  <property name="base_mass" value="4.0" />
-  <property name="shoulder_mass" value="3.7000" />
-  <property name="upper_arm_mass" value="8.3930" />
-  <property name="forearm_mass" value="2.2750" />
-  <property name="wrist_1_mass" value="1.2190" />
-  <property name="wrist_2_mass" value="1.2190" />
-  <property name="wrist_3_mass" value="0.1879" />
-  <property name="shoulder_cog" value="0.0 0.00193 -0.02561" />
-  <property name="upper_arm_cog" value="0.0 -0.024201 0.2125" />
-  <property name="forearm_cog" value="0.0 0.0265 0.11993" />
-  <property name="wrist_1_cog" value="0.0 0.110949 0.01634" />
-  <property name="wrist_2_cog" value="0.0 0.0018 0.11099" />
+<!-- Inertia parameters -->
+  <property name="base_mass" value="4.0" /> <!-- Invented number, only matters for simulator -->
+  <property name="shoulder_mass" value="7.778" />
+  <property name="upper_arm_mass" value="12.930" />
+  <property name="forearm_mass" value="3.87" />
+  <property name="wrist_1_mass" value="1.96" />
+  <property name="wrist_2_mass" value="1.96" />
+  <property name="wrist_3_mass" value="0.202" />
+  <!-- TODO -->
+  <property name="shoulder_cog" value="0.00008 0.00244 -0.037" />
+  <property name="upper_arm_cog" value="0.00008 0.00244   0.38757" />   <!-- 0.11336 - 0.089159 =  -->
+  <property name="forearm_cog" value="0.0 0.0265 0.11993" />       <!-- 0.119 is not half of 0.39225, is this really correct? -->
+  <property name="wrist_1_cog" value="0.0 0.110949 0.01634" />     <!-- 0.0018 + 0.10915 = 0.110949 -->
+  <property name="wrist_2_cog" value="0.0 0.0018 0.11099" />       <!-- 0.01634 + 0.09465 = 0.11099-->
   <property name="wrist_3_cog" value="0.0 0.001159 0.0" />
-  <!-- Kinematic model -->
-  <property name="shoulder_height" value="0.128" />
-  <property name="shoulder_offset" value="0.1704" />
-  <property name="upper_arm_length" value="0.60186" />
-  <property name="elbow_offset" value="0.12817" />
-  <property name="forearm_length" value="0.56415" />
-  <property name="wrist_1_length" value="0.11279" />
-  <property name="wrist_2_length" value="0.11279" />
-  <property name="wrist_3_length" value="0.0857" />
-  <property name="shoulder_radius" value="0.060" />
-  <property name="upper_arm_radius" value="0.054" />
-  <property name="elbow_radius" value="0.060" />
-  <property name="forearm_radius" value="0.040" />
-  <property name="wrist_radius" value="0.045" />
-  <!-- Collision model -->
-  <property name="base_collision_length" value="0.160" />
-  <property name="shoulder_collision_length" value="0.200" />
-  <property name="shoulder_collision_offset" value="0.035" />
-  <property name="elbow_collision_length" value="0.200" />
-  <property name="elbow_collision_offset" value="0.035" />
+  <!-- TODO -->
+<!-- Kinematic model -->
+  <property name="shoulder_height" value="0.1273" />
+  <property name="shoulder_offset" value="0.220941" />  <!-- shoulder_offset - elbow_offset + wrist_1_length = 0.220941 -->
+  <property name="upper_arm_length" value="0.612" />
+  <property name="elbow_offset" value="0.1719" />       <!-- CAD measured TODO -->
+  <property name="forearm_length" value="0.5723" />
+  <property name="wrist_1_length" value="0.1149" />     <!-- CAD measured TODO -->
+  <property name="wrist_2_length" value="0.1157" />
+  <property name="wrist_3_length" value="0.0922" />
+  <property name="shoulder_radius" value="0.075" />   <!-- manually measured -->
+  <property name="upper_arm_radius" value="0.054" />  <!-- manually measured -->
+  <property name="elbow_radius" value="0.060" />      <!-- manually measured -->
+  <property name="forearm_radius" value="0.043" />    <!-- manually measured -->
+  <property name="wrist_radius" value="0.045" />      <!-- manually measured -->
+<!-- Collision model -->
+  <property name="base_collision_length" value="0.215" />      <!-- manually measured -->
+  <property name="shoulder_collision_length" value="0.177" />  <!-- manually measured -->
+  <property name="shoulder_collision_offset" value="0.035" />  <!-- manually measured -->
+  <property name="elbow_collision_length" value="0.200" />     <!-- manually measured -->
+  <property name="elbow_collision_offset" value="0.035" />     <!-- manually measured -->
   <xacro:macro name="ur10_robot" params="prefix">
   <link name="${prefix}base_link" >
     <visual>
       <geometry>
-        <mesh filename="package://ur_description/meshes/ur10/visual/Base.stl" />
-      </geometry>
-      <origin xyz="0.0 0.0 0.003" rpy="0.0 0.0 ${3.0 * pi / 4.0}" />
-      <material name="UR/Blue" />
-    </visual>
-    <collision>
-      <geometry>
-        <mesh filename="package://ur_description/meshes/ur10/collision/Base.stl" />
-      </geometry>
-      <origin xyz="0.0 0.0 0.003" rpy="0.0 0.0 ${3.0 * pi / 4.0}" />
-    </collision>
+        <mesh filename="package://ur_description/meshes/ur10/visual/Base.dae" scale="0.001 0.001 0.001"/>
+      </geometry>
+      <origin xyz="0.0 0.0 0.0" rpy="${pi / 2.0} 0.0 0.0" />
+    </visual>
     <inertial>
       <mass value="${base_mass}" />
@@ -73,12 +88,13 @@
     <visual>
       <geometry>
-          <mesh filename="package://ur_description/meshes/ur10/visual/Shoulder.stl" />
-      </geometry>
-      <material name="UR/Grey" />
-    </visual>
-    <collision>
-      <geometry>
-        <mesh filename="package://ur_description/meshes/ur10/collision/Shoulder.stl" />
-      </geometry>
+        <mesh filename="package://ur_description/meshes/ur10/visual/Shoulder.dae" scale="0.001 0.001 0.001"/>
+      </geometry>
+      <origin xyz="0.0 0.0 -0.127" rpy="${pi / 2.0} 0.0 0.0" />
+    </visual>
+    <collision>
+      <geometry>
+        <cylinder length="${base_collision_length}" radius="${shoulder_radius}"/>
+      </geometry>
+      <origin xyz="0.0 0.0 ${-shoulder_height + (base_collision_length/2.0)}" rpy="0.0 0.0 0.0" />
     </collision>
     <inertial>
@@ -99,19 +115,48 @@
     <visual>
       <geometry>
-        <mesh filename="package://ur_description/meshes/ur10/visual/UpperArm.stl" />
-      </geometry>
-      <origin xyz="0.0 0.0 0.0" rpy="0.0 0.0 0.0" />
-      <material name="UR/Blue" />
-    </visual>
-    <collision>
-      <geometry>
-        <mesh filename="package://ur_description/meshes/ur10/collision/UpperArm.stl" />
-      </geometry>
-       <origin xyz="0.0 0.0 0.0" rpy="0.0 0.0 0.0" />
-    </collision>
+        <mesh filename="package://ur_description/meshes/ur10/visual/UpperArm.dae" scale="0.001 0.001 0.001"/>
+      </geometry>
+      <origin xyz="0.0 -0.221 -0.127" rpy="${pi / 2.0} -${0*pi / 2.0} 0.0" />
+    </visual>
     <inertial>
       <mass value="${upper_arm_mass}" />
       <inertia ixx="1.0" ixy="0.0" ixz="0.0" iyy="1.0" iyz="0.0" izz="1.0"/>
       <origin xyz="${upper_arm_cog}" rpy="0.0 0.0 0.0" />
+    </inertial>
+  </link>
+  <joint name="${prefix}upper_shoulder_joint" type="fixed">
+    <parent link="${prefix}upper_arm_link" />
+    <child link = "${prefix}upper_shoulder_link" />
+    <origin xyz="0.0 -0.046 0.0" rpy="${-pi/2.0} ${pi} 0.0" />
+  </joint>
+  <link name="${prefix}upper_shoulder_link">
+    <collision>
+      <geometry>
+        <cylinder length="0.175" radius="${shoulder_radius}"/>
+      </geometry>
+      <origin xyz="0.0 0.0 ${-(0.085-0.175/2.0)}" rpy="0.0 0.0 0.0" />
+    </collision>
+    <inertial>
+      <mass value="0" />
+      <inertia ixx="1.0" ixy="0.0" ixz="0.0" iyy="1.0" iyz="0.0" izz="1.0"/>
+      <origin xyz="0.0 0.0 0.0" rpy="0.0 0.0 0.0" />
+    </inertial>
+  </link>
+  <joint name="${prefix}upper_arm_middle_joint" type="fixed">
+    <parent link="${prefix}upper_arm_link" />
+    <child link = "${prefix}upper_arm_middle_link" />
+    <origin xyz="0.0 -0.046 ${0.45/2.0+0.17-shoulder_radius}" rpy="${-pi/2.0} ${pi} 0.0" />
+  </joint>
+  <link name="${prefix}upper_arm_middle_link">
+    <collision>
+      <geometry>
+          <cylinder length="0.45" radius="${0.105/2.0}"/>
+      </geometry>
+      <origin xyz="0.0 0.0 0.0" rpy="${pi/2.0} 0.0 0.0" />
+    </collision>
+    <inertial>
+      <mass value="0" />
+      <inertia ixx="1.0" ixy="0.0" ixz="0.0" iyy="1.0" iyz="0.0" izz="1.0"/>
+      <origin xyz="0.0 0.0 0.0" rpy="0.0 0.0 0.0" />
     </inertial>
   </link>
@@ -126,13 +171,14 @@
   <link name="${prefix}forearm_link">
     <visual>
-       <geometry>
-        <mesh filename="package://ur_description/meshes/ur10/visual/Forearm.stl" />
-      </geometry>
-      <material name="UR/Grey" />
-    </visual>
-    <collision>
-      <geometry>
-        <mesh filename="package://ur_description/meshes/ur10/collision/Forearm.stl" />
-      </geometry>
+      <geometry>
+        <mesh filename="package://ur_description/meshes/ur10/visual/Forearm.dae" scale="0.001 0.001 0.001"/>
+      </geometry>
+      <origin xyz="0.0 -0.049 -0.739" rpy="${pi / 2.0} 0.0 0.0" />
+    </visual>
+    <collision>
+      <geometry>
+          <cylinder length="0.26" radius="${0.12/2.0}"/>
+      </geometry>
+      <origin xyz="0.0 ${0.26/2.0-0.065} 0.0" rpy="${pi/2.0} 0.0 0.0" />
     </collision>
     <inertial>
@@ -142,6 +188,24 @@
     </inertial>
   </link>
+  <joint name="${prefix}forearm_middle_joint" type="fixed">
+    <parent link="${prefix}forearm_link" />
+    <child link = "${prefix}forearm_middle_link" />
+    <origin xyz="0.0 0.0 ${0.57-0.45/2.0-0.12/2.0+0.01}" rpy="0.0 0.0 0.0" />
+  </joint>
+  <link name="${prefix}forearm_middle_link">
+    <collision>
+      <geometry>
+          <cylinder length="0.45" radius="${forearm_radius}"/>
+      </geometry>
+      <origin xyz="0.0 0.0 0.0" rpy="0.0 0.0 0.0" />
+    </collision>
+    <inertial>
+      <mass value="0" />
+      <inertia ixx="1.0" ixy="0.0" ixz="0.0" iyy="1.0" iyz="0.0" izz="1.0"/>
+      <origin xyz="0.0 0.0 0.0" rpy="0.0 0.0 0.0" />
+    </inertial>
+  </link>
   <joint name="${prefix}wrist_1_joint" type="revolute">
-     <parent link="${prefix}forearm_link" />
+    <parent link="${prefix}forearm_link" />
     <child link = "${prefix}wrist_1_link" />
     <origin xyz="0.0 0.0 ${forearm_length}" rpy="0.0 ${pi / 2.0} 0.0" />
@@ -153,14 +217,13 @@
     <visual>
       <geometry>
-        <mesh filename="package://ur_description/meshes/ur10/visual/Wrist1.stl" />
-      </geometry>
-      <origin xyz="0.0 ${wrist_1_length} 0.0" rpy="0.0 0 0.0" />
-      <material name="UR/Blue" />
-    </visual>
-    <collision>
-      <geometry>
-        <mesh filename="package://ur_description/meshes/ur10/collision/Wrist1.stl" />
-      </geometry>
-      <origin xyz="0.0 ${wrist_1_length} 0.0" rpy="0.0 0 0.0" />
+        <mesh filename="package://ur_description/meshes/ur10/visual/Wrist1.dae" scale="0.001 0.001 0.001"/>
+      </geometry>
+      <origin xyz="0.0 -0.049 -1.312" rpy="${pi / 2.0} 0.0 0.0" />
+    </visual>
+    <collision>
+      <geometry>
+        <cylinder length="${0.123}" radius="${wrist_radius}"/>
+      </geometry>
+      <origin xyz="0.0 ${0.123/2.0-0.057} 0.0" rpy="${-pi/2.0} 0.0 0.0" />
     </collision>
     <inertial>
@@ -170,5 +233,5 @@
     </inertial>
   </link>
-    <joint name="${prefix}wrist_2_joint" type="revolute">
+  <joint name="${prefix}wrist_2_joint" type="revolute">
     <parent link="${prefix}wrist_1_link" />
     <child link = "${prefix}wrist_2_link" />
@@ -181,14 +244,13 @@
     <visual>
       <geometry>
-        <mesh filename="package://ur_description/meshes/ur10/visual/Wrist2.stl" />
-      </geometry>
-      <origin xyz="0.0 0.0 ${wrist_2_length}" rpy="0.0 0.0 0.0" />
-      <material name="UR/Grey" />
-    </visual>
-    <collision>
-      <geometry>
-        <mesh filename="package://ur_description/meshes/ur10/collision/Wrist2.stl" />
-      </geometry>
-      <origin xyz="0.0 0.0 ${wrist_2_length}" rpy="0.0 0.0 0.0" />
+        <mesh filename="package://ur_description/meshes/ur10/visual/Wrist2.dae" scale="0.001 0.001 0.001"/>
+      </geometry>
+      <origin xyz="0.0 -0.164 -1.312" rpy="${pi / 2.0} 0.0 0.0" />
+    </visual>
+    <collision>
+      <geometry>
+        <cylinder length="0.123" radius="${wrist_radius}"/>
+      </geometry>
+      <origin xyz="0.0 0.0 ${0.123/2.0-0.057}" rpy="0.0 0.0 0.0" />
     </collision>
     <inertial>
@@ -209,21 +271,26 @@
     <visual>
       <geometry>
-        <mesh filename="package://ur_description/meshes/ur10/visual/Wrist3.stl" />
-      </geometry>
-       <origin xyz="0.0 ${wrist_3_length} 0.0" rpy="0.0 0.0 0" />
-      <material name="UR/Blue" />
-    </visual>
-    <collision>
-      <geometry>
-        <mesh filename="package://ur_description/meshes/ur10/collision/Wrist3.stl" />
-      </geometry>
-      <origin xyz="0.0 ${wrist_3_length} 0.0" rpy="0.0 0.0 0" />
-    </collision>
-    <inertial>
-       <mass value="${wrist_3_mass}" />
+        <mesh filename="package://ur_description/meshes/ur10/visual/Wrist3.dae" scale="0.001 0.001 0.001"/>
+      </geometry>
+      <origin xyz="0.0 -0.164 -1.427" rpy="${pi / 2.0} 0.0 0.0" />
+    </visual>
+    <collision>
+      <geometry>
+          <cylinder length="${0.123+0.025}" radius="${wrist_radius}"/>
+      </geometry>
+      <origin xyz="0.0 ${(0.123+0.025)/2.0-0.057} 0.0" rpy="${-pi/2.0} 0.0 0.0" />
+    </collision>
+    <inertial>
+      <mass value="${wrist_3_mass}" />
       <origin xyz="${wrist_3_cog}" rpy="0.0 0.0 0.0" />
       <inertia ixx="1.0" ixy="0.0" ixz="0.0" iyy="1.0" iyz="0.0" izz="1.0"/>
     </inertial>
   </link>
+  <joint name="${prefix}ee_fixed_joint" type="fixed">
+    <parent link="${prefix}wrist_3_link" />
+    <child link = "${prefix}ee_link" />
+    <origin xyz="0.0 ${wrist_3_length} 0.0" rpy="0.0 0.0 ${pi/2.0}" />
+  </joint>
+  <link name="${prefix}ee_link" />
   <xacro:ur10_arm_transmission prefix="${prefix}" />
   <xacro:ur10_arm_gazebo prefix="${prefix}" />

Commit message: added collision model for ur10 base

File: ur_description/urdf/ur10.urdf.xacro (robot description, xacro)
@@ -72,4 +72,10 @@
       <origin xyz="0.0 0.0 0.0" rpy="${pi / 2.0} 0.0 0.0" />
     </visual>
+    <collision>
+      <geometry>
+        <cylinder length="${0.04}" radius="${shoulder_radius+0.03}"/>
+      </geometry>
+      <origin xyz="0.0 0.0 0.02" rpy="0.0 0.0 0.0" />
+    </collision>
     <inertial>
       <mass value="${base_mass}" />

Commit message: introduced cylinder macro

File: ur_description/urdf/ur10.urdf.xacro (robot description, xacro)
@@ -7,4 +7,7 @@
   <include filename="$(find ur_description)/urdf/ur10.gazebo.xacro" />
   <include filename="$(find ur_description)/urdf/materials.urdf.xacro" />
+  <xacro:macro name="cylinder_model" params="length radius">
+    <cylinder length="${length}" radius="${radius}"/>
+  </xacro:macro>
 <!--
 DH for UR5:
@@ -74,5 +77,5 @@
     <collision>
       <geometry>
-        <cylinder length="${0.04}" radius="${shoulder_radius+0.03}"/>
+        <xacro:cylinder_model length="${0.04}" radius="${shoulder_radius+0.03}"/>
       </geometry>
       <origin xyz="0.0 0.0 0.02" rpy="0.0 0.0 0.0" />
@@ -100,5 +103,5 @@
     <collision>
       <geometry>
-        <cylinder length="${base_collision_length}" radius="${shoulder_radius}"/>
+        <xacro:cylinder_model length="${base_collision_length}" radius="${shoulder_radius}"/>
       </geometry>
       <origin xyz="0.0 0.0 ${-shoulder_height + (base_collision_length/2.0)}" rpy="0.0 0.0 0.0" />
@@ -139,5 +142,5 @@
     <collision>
       <geometry>
-        <cylinder length="0.175" radius="${shoulder_radius}"/>
+        <xacro:cylinder_model length="0.175" radius="${shoulder_radius}"/>
       </geometry>
       <origin xyz="0.0 0.0 ${-(0.085-0.175/2.0)}" rpy="0.0 0.0 0.0" />
@@ -157,5 +160,5 @@
     <collision>
       <geometry>
-          <cylinder length="0.45" radius="${0.105/2.0}"/>
+          <xacro:cylinder_model length="0.45" radius="${0.105/2.0}"/>
       </geometry>
       <origin xyz="0.0 0.0 0.0" rpy="${pi/2.0} 0.0 0.0" />
@@ -184,5 +187,5 @@
     <collision>
       <geometry>
-          <cylinder length="0.26" radius="${0.12/2.0}"/>
+          <xacro:cylinder_model length="0.26" radius="${0.12/2.0}"/>
       </geometry>
       <origin xyz="0.0 ${0.26/2.0-0.065} 0.0" rpy="${pi/2.0} 0.0 0.0" />
@@ -202,5 +205,5 @@
     <collision>
       <geometry>
-          <cylinder length="0.45" radius="${forearm_radius}"/>
+          <xacro:cylinder_model length="0.45" radius="${forearm_radius}"/>
       </geometry>
       <origin xyz="0.0 0.0 0.0" rpy="0.0 0.0 0.0" />
@@ -229,5 +232,5 @@
     <collision>
       <geometry>
-        <cylinder length="${0.123}" radius="${wrist_radius}"/>
+        <xacro:cylinder_model length="${0.123}" radius="${wrist_radius}"/>
       </geometry>
       <origin xyz="0.0 ${0.123/2.0-0.057} 0.0" rpy="${-pi/2.0} 0.0 0.0" />
@@ -256,5 +259,5 @@
     <collision>
       <geometry>
-        <cylinder length="0.123" radius="${wrist_radius}"/>
+        <xacro:cylinder_model length="0.123" radius="${wrist_radius}"/>
       </geometry>
       <origin xyz="0.0 0.0 ${0.123/2.0-0.057}" rpy="0.0 0.0 0.0" />
@@ -283,5 +286,5 @@
     <collision>
       <geometry>
-          <cylinder length="${0.123+0.025}" radius="${wrist_radius}"/>
+          <xacro:cylinder_model length="${0.123+0.025}" radius="${wrist_radius}"/>
       </geometry>
       <origin xyz="0.0 ${(0.123+0.025)/2.0-0.057} 0.0" rpy="${-pi/2.0} 0.0 0.0" />

Commit message: xacro properties for default joint limits

File: ur_description/urdf/ur10.urdf.xacro (robot description, xacro)
@@ -8,5 +8,6 @@
   <include filename="$(find ur_description)/urdf/materials.urdf.xacro" />
   <xacro:macro name="cylinder_model" params="length radius">
-    <cylinder length="${length}" radius="${radius}"/>
+    <!--<cylinder length="${length}" radius="${radius}"/> -->
+    <mesh filename="package://ur_description/meshes/unit_cyl.stl" scale="${radius} ${radius} ${length}"/>
   </xacro:macro>
 <!--
@@ -67,4 +68,8 @@
   <property name="elbow_collision_length" value="0.200" />     <!-- manually measured -->
   <property name="elbow_collision_offset" value="0.035" />     <!-- manually measured -->
+  <property name="joint_limit_lower" value="${-2.0 * pi}" />
+  <property name="joint_limit_upper" value="${2.0 * pi}" />
+  <property name="joint_limit_effort" value="10.0" />
+  <property name="joint_limit_velocity" value="${pi}" />
   <xacro:macro name="ur10_robot" params="prefix">
   <link name="${prefix}base_link" >
@@ -91,5 +96,5 @@
     <origin xyz="0.0 0.0 ${shoulder_height}" rpy="0.0 0.0 0.0" />
     <axis xyz="0.0 0.0 1.0" />
-    <limit lower="${-2.0 * pi}" upper="${2.0 * pi}" effort="10.0" velocity="${pi}"/>
+    <limit lower="${joint_limit_lower}" upper="${joint_limit_upper}" effort="${joint_limit_effort}" velocity="${joint_limit_velocity}"/>
     <dynamics damping="10" friction="0.1"/>
   </joint>
@@ -118,5 +123,5 @@
     <origin xyz="0.0 ${shoulder_offset} 0.0" rpy="0.0 ${pi / 2.0} 0.0" />
     <axis xyz="0.0 1.0 0.0" />
-    <limit lower="${-2.0 * pi}" upper="${2.0 * pi}" effort="10.0" velocity="${pi}"/>
+    <limit lower="${joint_limit_lower}" upper="${joint_limit_upper}" effort="${joint_limit_effort}" velocity="${joint_limit_velocity}"/>
     <dynamics damping="10" friction="0.1"/>
   </joint>
@@ -175,5 +180,5 @@
     <origin xyz="0.0 ${-elbow_offset} ${upper_arm_length}" rpy="0.0 0.0 0.0" />
     <axis xyz="0.0 1.0 0.0" />
-    <limit lower="${-2.0 * pi}" upper="${2.0 * pi}" effort="10.0" velocity="${pi}"/>
+    <limit lower="${joint_limit_lower}" upper="${joint_limit_upper}" effort="${joint_limit_effort}" velocity="${joint_limit_velocity}"/>
     <dynamics damping="10" friction="0.1"/>
   </joint>
@@ -220,5 +225,5 @@
     <origin xyz="0.0 0.0 ${forearm_length}" rpy="0.0 ${pi / 2.0} 0.0" />
     <axis xyz="0.0 1.0 0.0" />
-    <limit lower="${-2.0 * pi}" upper="${2.0 * pi}" effort="10.0" velocity="${pi}"/>
+    <limit lower="${joint_limit_lower}" upper="${joint_limit_upper}" effort="${joint_limit_effort}" velocity="${joint_limit_velocity}"/>
     <dynamics damping="10" friction="0.1"/>
   </joint>
@@ -247,5 +252,5 @@
     <origin xyz="0.0 ${wrist_1_length} 0.0" rpy="0.0 0.0 0.0" />
     <axis xyz="0.0 0.0 1.0" />
-    <limit lower="${-2.0 * pi}" upper="${2.0 * pi}" effort="10.0" velocity="${pi}"/>
+    <limit lower="${joint_limit_lower}" upper="${joint_limit_upper}" effort="${joint_limit_effort}" velocity="${joint_limit_velocity}"/>
     <dynamics damping="10" friction="0.1"/>
   </joint>
@@ -274,5 +279,5 @@
     <origin xyz="0.0 0.0 ${wrist_2_length}" rpy="0.0 0.0 0.0" />
     <axis xyz="0.0 1.0 0.0" />
-    <limit lower="${-2.0 * pi}" upper="${2.0 * pi}" effort="10.0" velocity="${pi}"/>
+    <limit lower="${joint_limit_lower}" upper="${joint_limit_upper}" effort="${joint_limit_effort}" velocity="${joint_limit_velocity}"/>
     <dynamics damping="10" friction="0.1"/>
   </joint>
