Commit message: increased damping to 1000

File: ur_description/urdf/ur10.urdf.xacro (robot description, xacro)
@@ -97,5 +97,5 @@
     <axis xyz="0.0 0.0 1.0" />
     <limit lower="${joint_limit_lower}" upper="${joint_limit_upper}" effort="${joint_limit_effort}" velocity="${joint_limit_velocity}"/>
-    <dynamics damping="10" friction="0.1"/>
+    <dynamics damping="1000" friction="0.1"/>
   </joint>
   <link name="${prefix}shoulder_link">
@@ -124,5 +124,5 @@
     <axis xyz="0.0 1.0 0.0" />
     <limit lower="${joint_limit_lower}" upper="${joint_limit_upper}" effort="${joint_limit_effort}" velocity="${joint_limit_velocity}"/>
-    <dynamics damping="10" friction="0.1"/>
+    <dynamics damping="1000" friction="0.1"/>
   </joint>
   <link name="${prefix}upper_arm_link">
@@ -181,5 +181,5 @@
     <axis xyz="0.0 1.0 0.0" />
     <limit lower="${joint_limit_lower}" upper="${joint_limit_upper}" effort="${joint_limit_effort}" velocity="${joint_limit_velocity}"/>
-    <dynamics damping="10" friction="0.1"/>
+    <dynamics damping="1000" friction="0.1"/>
   </joint>
   <link name="${prefix}forearm_link">
@@ -226,5 +226,5 @@
     <axis xyz="0.0 1.0 0.0" />
     <limit lower="${joint_limit_lower}" upper="${joint_limit_upper}" effort="${joint_limit_effort}" velocity="${joint_limit_velocity}"/>
-    <dynamics damping="10" friction="0.1"/>
+    <dynamics damping="1000" friction="0.1"/>
   </joint>
   <link name="${prefix}wrist_1_link">
@@ -253,5 +253,5 @@
     <axis xyz="0.0 0.0 1.0" />
     <limit lower="${joint_limit_lower}" upper="${joint_limit_upper}" effort="${joint_limit_effort}" velocity="${joint_limit_velocity}"/>
-    <dynamics damping="10" friction="0.1"/>
+    <dynamics damping="1000" friction="0.1"/>
   </joint>
   <link name="${prefix}wrist_2_link">
@@ -280,5 +280,5 @@
     <axis xyz="0.0 1.0 0.0" />
     <limit lower="${joint_limit_lower}" upper="${joint_limit_upper}" effort="${joint_limit_effort}" velocity="${joint_limit_velocity}"/>
-    <dynamics damping="10" friction="0.1"/>
+    <dynamics damping="1000" friction="0.1"/>
   </joint>
   <link name="${prefix}wrist_3_link">
